File: indicator_module/indicator_module.kicad_pcb (KiCad board)
At the start: 2 copper layers, 47.1 x 30.9 mm, 31 parts, among them J1 BUS_A, J2 BUS_B

Commit message: Relabel nand/indicator board FETs BSS -> AO34xxA (value text only)
AO3400A/AO3401A are pin-compatible SOT-23 drop-ins for BSS138/BSS84, so only
the silkscreen Value changes. Routing (nand: 211 segments, 29 vias, GND zone),
placement and labels untouched. Boards verified to load in pcbnew.
Parts:
- NAND_1_QA, NAND_1_QB, NAND_1_QY, NAND_2_QA, NAND_2_QB, NAND_2_QY, NAND_3_QA, NAND_3_QB, NAND_3_QY, NAND_4_QA, NAND_4_QB, NAND_4_QY: value BSS138 -> AO3400A
Changed lines of the file:
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@@
 			)
 		)
-		(property "Value" "BSS138"
+		(property "Value" "AO3400A"
 			(at 0 2.4 0)
 			(layer "F.Fab")
@@
 			)
 		)
-		(property "Value" "BSS138"
+		(property "Value" "AO3400A"
 			(at 0 2.4 0)
 			(layer "F.Fab")
@@
 			)
 		)
-		(property "Value" "BSS138"
+		(property "Value" "AO3400A"
 			(at 0 2.4 0)
 			(layer "F.Fab")
@@
 			)
 		)
-		(property "Value" "BSS138"
+		(property "Value" "AO3400A"
 			(at 0 2.4 0)
 			(layer "F.Fab")
@@
 			)
 		)
-		(property "Value" "BSS138"
+		(property "Value" "AO3400A"
 			(at 0 2.4 0)
 			(layer "F.Fab")
@@
 			)
 		)
-		(property "Value" "BSS138"
+		(property "Value" "AO3400A"
 			(at 0 2.4 0)
 			(layer "F.Fab")
@@
 			)
 		)
-		(property "Value" "BSS138"
+		(property "Value" "AO3400A"
 			(at 0 2.4 0)
 			(layer "F.Fab")
@@
 			)
 		)
-		(property "Value" "BSS138"
+		(property "Value" "AO3400A"
 			(at 0 2.4 0)
 			(layer "F.Fab")
@@
 			)
 		)
-		(property "Value" "BSS138"
+		(property "Value" "AO3400A"
 			(at 0 2.4 0)
 			(layer "F.Fab")
@@
 			)
 		)
-		(property "Value" "BSS138"
+		(property "Value" "AO3400A"
 			(at 0 2.4 0)
 			(layer "F.Fab")
@@
 			)
 		)
-		(property "Value" "BSS138"
+		(property "Value" "AO3400A"
 			(at 0 2.4 0)
 			(layer "F.Fab")
@@
 			)
 		)
-		(property "Value" "BSS138"
+		(property "Value" "AO3400A"
 			(at 0 2.4 0)
 			(layer "F.Fab")

Commit message: Regenerate indicator board from current netlist
Was stale (NAND_* nets, NAND_n_QA refs, BSS138). Now SIG1..SIG12 nets,
D1..D12 / Q1..Q12 refs, AO3400A. Unrouted board, no manual work lost.
Parts:
- removed NAND_1_A: NAND_1_A, LED_SMD:LED_0805_2012Metric
- removed NAND_1_B: NAND_1_B, LED_SMD:LED_0805_2012Metric
- removed NAND_1_QA, NAND_1_QB, NAND_1_QY, NAND_2_QA, NAND_2_QB, NAND_2_QY, NAND_3_QA, NAND_3_QB, NAND_3_QY, NAND_4_QA, NAND_4_QB, NAND_4_QY: AO3400A, Package_TO_SOT_SMD:SOT-23
- removed NAND_1_Y: NAND_1_Y, LED_SMD:LED_0805_2012Metric
- removed NAND_2_A: NAND_2_A, LED_SMD:LED_0805_2012Metric
- removed NAND_2_B: NAND_2_B, LED_SMD:LED_0805_2012Metric
- removed NAND_2_Y: NAND_2_Y, LED_SMD:LED_0805_2012Metric
- removed NAND_3_A: NAND_3_A, LED_SMD:LED_0805_2012Metric
- removed NAND_3_B: NAND_3_B, LED_SMD:LED_0805_2012Metric
- removed NAND_3_Y: NAND_3_Y, LED_SMD:LED_0805_2012Metric
- removed NAND_4_A: NAND_4_A, LED_SMD:LED_0805_2012Metric
- removed NAND_4_B: NAND_4_B, LED_SMD:LED_0805_2012Metric
- removed NAND_4_Y: NAND_4_Y, LED_SMD:LED_0805_2012Metric
- added D1: D1, LED_SMD:LED_0805_2012Metric, F.Cu at (22.4, 29.0)
- added D10: D10, LED_SMD:LED_0805_2012Metric, F.Cu at (50.9, 29.0)
- added D11: D11, LED_SMD:LED_0805_2012Metric, F.Cu at (50.9, 33.5)
- added D12: D12, LED_SMD:LED_0805_2012Metric, F.Cu at (50.9, 38.0)
- added D2: D2, LED_SMD:LED_0805_2012Metric, F.Cu at (22.4, 33.5)
- added D3: D3, LED_SMD:LED_0805_2012Metric, F.Cu at (22.4, 38.0)
- added D4: D4, LED_SMD:LED_0805_2012Metric, F.Cu at (31.9, 29.0)
- added D5: D5, LED_SMD:LED_0805_2012Metric, F.Cu at (31.9, 33.5)
- added D6: D6, LED_SMD:LED_0805_2012Metric, F.Cu at (31.9, 38.0)
- added D7: D7, LED_SMD:LED_0805_2012Metric, F.Cu at (41.4, 29.0)
- added D8: D8, LED_SMD:LED_0805_2012Metric, F.Cu at (41.4, 33.5)
- added D9: D9, LED_SMD:LED_0805_2012Metric, F.Cu at (41.4, 38.0)
- added Q1: AO3400A, Package_TO_SOT_SMD:SOT-23, F.Cu at (27.2, 29.0)
- added Q10: AO3400A, Package_TO_SOT_SMD:SOT-23, F.Cu at (55.7, 29.0)
- added Q11: AO3400A, Package_TO_SOT_SMD:SOT-23, F.Cu at (55.7, 33.5)
- added Q12: AO3400A, Package_TO_SOT_SMD:SOT-23, F.Cu at (55.7, 38.0)
- added Q2: AO3400A, Package_TO_SOT_SMD:SOT-23, F.Cu at (27.2, 33.5)
- added Q3: AO3400A, Package_TO_SOT_SMD:SOT-23, F.Cu at (27.2, 38.0)
- added Q4: AO3400A, Package_TO_SOT_SMD:SOT-23, F.Cu at (36.7, 29.0)
- added Q5: AO3400A, Package_TO_SOT_SMD:SOT-23, F.Cu at (36.7, 33.5)
- added Q6: AO3400A, Package_TO_SOT_SMD:SOT-23, F.Cu at (36.7, 38.0)
- added Q7: AO3400A, Package_TO_SOT_SMD:SOT-23, F.Cu at (46.2, 29.0)
- added Q8: AO3400A, Package_TO_SOT_SMD:SOT-23, F.Cu at (46.2, 33.5)
- added Q9: AO3400A, Package_TO_SOT_SMD:SOT-23, F.Cu at (46.2, 38.0)
- J1: value BUS_A -> BUS_STACK_1x16
- J2: value BUS_B -> BUS_STACK_1x16
Connections:
- net NAND_1_A renamed SIG1
- net NAND_1_B renamed SIG2
- net NAND_1_Y renamed SIG3
- net NAND_2_A renamed SIG4
- net NAND_2_B renamed SIG5
- net NAND_2_Y renamed SIG6
- net NAND_3_A renamed SIG7
- net NAND_3_B renamed SIG8
- net NAND_3_Y renamed SIG9
- net NAND_4_A renamed SIG10
- net NAND_4_B renamed SIG11
- net NAND_4_Y renamed SIG12
Routing:
- added copper zone on B.Cu, net GND
